File: DigitalDC.kicad_sch (KiCad schematic)
At the start: 24 parts, among them J1 Conn_01x08_Pin, U1 LM358, U2 MT3608, U3 MCP4801

Commit message: Version 1 is done
Parts:
- added D3: GRN, LED_SMD:LED_0805_2012Metric_Pad1.15x1.40mm_HandSolder, symbol Device:LED
- added R10, R11: 0, Resistor_SMD:R_0603_1608Metric_Pad0.98x0.95mm_HandSolder, symbol Device:R
- added R12: 1k, Resistor_SMD:R_0603_1608Metric_Pad0.98x0.95mm_HandSolder, symbol Device:R
- added TP1: GND, TestPoint:TestPoint_Bridge_Pitch2.54mm_Drill1.0mm, symbol Connector:TestPoint
- added TP7: TestPoint, TestPoint:TestPoint_Pad_1.5x1.5mm, symbol Connector:TestPoint
- C1: footprint (none) -> Capacitor_SMD:C_0603_1608Metric_Pad1.08x0.95mm_HandSolder
- C2: footprint (none) -> Capacitor_SMD:C_1210_3225Metric_Pad1.33x2.70mm_HandSolder
- C3, C4: value C -> 0.1; footprint (none) -> Capacitor_SMD:C_0603_1608Metric_Pad1.08x0.95mm_HandSolder
- D2: value LED -> YEL; footprint (none) -> LED_SMD:LED_0805_2012Metric_Pad1.15x1.40mm_HandSolder
- J1: footprint (none) -> Connector_PinHeader_2.54mm:PinHeader_1x08_P2.54mm_Vertical
- L1: footprint (none) -> Inductor_SMD:L_Taiyo-Yuden_NR-30xx_HandSoldering
- R1, R2, R3, R4, R5, R6, R7, R8, R9: footprint (none) -> Resistor_SMD:R_0603_1608Metric_Pad0.98x0.95mm_HandSolder
- TP2: renamed from TP1; value TestPoint -> DAC; footprint (none) -> TestPoint:TestPoint_Bridge_Pitch2.54mm_Drill1.0mm
- TP3: renamed from TP4; value TestPoint -> FB; footprint (none) -> TestPoint:TestPoint_Bridge_Pitch2.54mm_Drill1.0mm
- TP4: renamed from TP2; value TestPoint -> V reg; footprint (none) -> TestPoint:TestPoint_Bridge_Pitch2.54mm_Drill1.0mm
- TP5: renamed from TP3; value TestPoint -> V Out; footprint (none) -> TestPoint:TestPoint_Bridge_Pitch2.54mm_Drill1.0mm
- U1, U3: footprint (none) -> Package_SO:SOIC-8_3.9x4.9mm_P1.27mm
Connections:
- net +5V: now also D3.2 (A)
- net GND: now also R10.2, R11.2, R12.2, TP1.1
- net at R8.2, U3.6 (~{SHDN}): now also J1.6 (Pin_6); no longer J1.3 (Pin_3)
- net at R7.2, R9.1, U3.5 (~{LDAC}): now also J1.7 (Pin_7); no longer J1.4 (Pin_4)
- net at U3.2 (~{CS}): now also J1.3 (Pin_3); no longer J1.5 (Pin_5)
- net at U3.3 (SCK): now also J1.4 (Pin_4); no longer J1.6 (Pin_6)
- net at U3.4 (SDI): now also J1.5 (Pin_5); no longer J1.7 (Pin_7)
- net at U1.1: now also TP7.1
- net at U1.2 (-): now also R10.1
- net at U1.3 (+): now also R11.1
- new net: D3.1 (K), R12.1
Other:
- moved on the sheet: J1, U1A
